File: hardware/function_power_input.kicad_sch (KiCad schematic)
At the start: 17 parts, among them J5 Conn_01x03_Socket, J6 Conn_01x03_Socket, U2 AZ1117-3.3

Commit message: auto updated
Parts:
- removed R2: 0, Resistor_SMD:R_0805_2012Metric, symbol Device:R
- renumbered C13 to C15, C14 to C16, D1 to D4, D4 to D5, D2 to D6, D3 to D7, R28 to R21, R26 to R22, R27 to R23, TP1 to TP5, TP2 to TP6, TP3 to TP7, U2 to U3
Connections:
- net +3.3V: now also C16.1, TP6.1, U3.2 (VO)
Other:
- note added: "required by the usb standard"

Commit message: added more ground testpoint for osc prob clip and status led for vbus
Parts:
- added D8: LED, LED_SMD:LED_0805_2012Metric, symbol Device:LED
- added R31: 300, Resistor_SMD:R_0805_2012Metric, symbol Device:R
- added TP8, TP9: GND, TestPoint:TestPoint_Bridge_Pitch2.54mm_Drill0.7mm, symbol Connector:TestPoint
- J6: footprint Connector_Molex:Molex_KK-396_A-41791-0003_1x03_P3.96mm_Vertical -> Connector_PinSocket_2.54mm:PinSocket_1x03_P2.54mm_Vertical
Connections:
- net GND: now also D8.1 (K), TP8.1, TP9.1
- net VBUS: now also R31.2
- new net: D8.2 (A), R31.1
Other:
- moved on the sheet: TP7
