File: hardware/function_amplifier.kicad_sch (KiCad schematic)
At the start: 24 parts, among them J7 pre_amp, U3 TL074

Commit message: auto updated
Parts:
- renumbered C15 to C13, C16 to C14, J7 to J4, R15 to R10, R16 to R11, R17 to R12, R18 to R13, R19 to R14, R20 to R15, R21 to R16, R22 to R17, R23 to R18, R24 to R19, R25 to R20, R10 to R5, R11 to R6, R12 to R7, R13 to R8, R14 to R9, TP4 to TP1, TP5 to TP2, TP6 to TP3, TP7 to TP4, U3 to U2

Commit message: updated
Connections:
- net CH1_OUT: now also U2.8; no longer U2.1
- net CH2_OUT: now also U2.7; no longer U2.8
- net CH3_OUT: now also U2.14; no longer U2.7
- net CH4_OUT: now also U2.1; no longer U2.14
- net at R14.2, R17.2: now also U2.5 (+); no longer U2.10 (+)
- net at R11.1, R5.2: now also U2.9 (-); no longer U2.2 (-)
- net at R6.2, R9.2: now also U2.10 (+); no longer U2.3 (+)
- net at R12.1, R7.2: now also U2.13 (-); no longer U2.6 (-)
- net at R16.2, R18.2: now also U2.3 (+); no longer U2.12 (+)
- net at R15.2, R20.1: now also U2.2 (-); no longer U2.13 (-)
- net at R10.2, R8.2: now also U2.12 (+); no longer U2.5 (+)
- net at R13.2, R19.1: now also U2.6 (-); no longer U2.9 (-)
Other:
- moved on the sheet: U2A, U2B, U2C, U2D
