File: hardware/function_gen.kicad_pcb (KiCad board)
At the start: 4 copper layers, 71 x 60.9 mm, 94 parts, among them J1 Conn_01x01, J10 Conn_01x01, J11 Conn_01x01, J2 Conn_ARM_SWD_TagConnect_TC203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, J3 Conn_01x08, J5 Conn_01x03_Socket, J6 Conn_01x03_Socket, J7 USB_C_Receptacle_USB2.0, J8 Conn_01x05_Pin, J9 Conn_01x05_Pin, SW1 SW_SPDT, SW2 SW_Push, SW3 SW_SP4T, SW4 SW_SP4T, SW5 SW_SP4T, SW6 SW_SP4T, SW7 SW_SPST, SW8 SW_SPST, U1 STM32G431CBTx, U2 TL074, U3 AZ1117-3.3, Y1 Crystal_GND24

Commit message: complete redesgin
Parts:
- removed D2, D3: LED, LED_SMD:LED_0805_2012Metric
- removed J1, J10, J11: Conn_01x01, TestPoint:TestPoint_Pad_1.0x1.0mm
- removed R1: 10k, Resistor_SMD:R_0805_2012Metric
- added D10: LED, LED_SMD:LED_0805_2012Metric, F.Cu at (141.3, 90.9)
- added D11: LED, LED_SMD:LED_0805_2012Metric, F.Cu at (141.3, 96.1)
- added D12: LED, LED_SMD:LED_0805_2012Metric, F.Cu at (141.1, 101.6)
- added D9: LED, LED_SMD:LED_0805_2012Metric, F.Cu at (141.3, 85.4)
- added R32: 500, Resistor_SMD:R_0805_2012Metric, B.Cu at (143.2, 85.4)
- added R33: 500, Resistor_SMD:R_0805_2012Metric, B.Cu at (143.2, 91.5)
- added R34: 500, Resistor_SMD:R_0805_2012Metric, B.Cu at (143.2, 96.1)
- added R35: 500, Resistor_SMD:R_0805_2012Metric, B.Cu at (143.0, 101.6)
- J8, J9: footprint Connector_PinHeader_2.54mm:PinHeader_1x05_P2.54mm_Vertical -> Connector_JST:JST_XH_B5B-XH-AM_1x05_P2.50mm_Vertical
- moved SW1 56.9 mm to (70.0, 100.2)
- moved J2 50.1 mm to (70.4, 114.1), turned to 90 degrees
- moved U1 19.6 mm to (129.2, 72.2)
- moved J9 11.3 mm to (111.6, 93.3), turned to 90 degrees
- moved C4 1.19 mm to (138.6, 97.3), turned to -45 degrees
- moved J8 1.11 mm to (111.6, 109.4), turned to 90 degrees
- moved G*** 0.68 mm to (131.6, 58.3)
- moved C1 0.58 mm to (132.8, 101.4), turned to 135 degrees
- turned Y1 to 135 degrees
- renumbered TPGND to TP8
Routing:
- net /NRST: track 47.3 -> 2.75 mm, vias 3 -> 0
- net GND: track 94.3 -> 53.2 mm, vias 47 -> 31
- net /I2S3_SD: track 21.9 -> 0.00 mm
- net /I2S3_CK-SWO: track 20.2 -> 0.00 mm, vias 1 -> 0
- net /USART3_CK: track 20.1 -> 0.00 mm, vias 1 -> 0
- net /OPAMP3_VOUT: track 30.6 -> 11.1 mm
- net /I2S3_WS: track 18.9 -> 0.00 mm
- net /GPIO_4: track 0.00 -> 18.0 mm, vias 0 -> 2
- net /OPAMP1_VOUT: track 38.7 -> 22.1 mm
- net /ADC2_IN3: track 24.1 -> 8.13 mm
- net /USB_D+: track 21.9 -> 6.93 mm
- net /USB_D-: track 21.2 -> 6.39 mm
- net /SW_DIO: track 14.7 -> 0.00 mm
- net /ADC2_IN12: track 51.5 -> 37.1 mm
- net /UCPD1_CC1: track 29.3 -> 15.0 mm
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Other:
- outline, holes or cut-outs redrawn
- board text added: "CK"
- board text added: "REV3-pending"
- board text added: "RX"
- board text added: "TX"
- board text added: "have you touched grass today"
- board text removed: "IO1"
- board text removed: "IO2"
- board text removed: "IO3"
- board text removed: "REV2-1"
- board text removed: "USART_CK"
- board text removed: "USART_RX"
- board text removed: "USART_TX"

Commit message: updated
Parts:
- removed the C8 at (139.9, 110.2)
- removed the C8 at (130.1, 85.4)
- removed the G*** at (131.6, 58.3)
- removed the G*** at (130.3, 91.8)
- removed R34, R35: 500, Resistor_SMD:R_0805_2012Metric
- removed TP3, TP4: TestPoint, TestPoint:TestPoint_Pad_D1.5mm
- removed TP7: GND, TestPoint:TestPoint_Pad_D1.5mm
- added ?: , , F.Cu at (115.8, 74.4)
- added ?: , , F.Cu at (115.8, 125.4)
- added ?: , , F.Cu at (141.2, 125.4)
- added ?: , , F.Cu at (167.6, 74.4)
- added ?: , , F.Cu at (174.8, 125.4)
- added A: TestPoint, TestPoint:TestPoint_Pad_D1.5mm, F.Cu at (119.4, 107.9)
- added B: TestPoint, TestPoint:TestPoint_Pad_D1.5mm, F.Cu at (125.3, 107.9)
- added C12: 100n, Capacitor_SMD:C_0805_2012Metric, B.Cu at (114.5, 96.1)
- added C17: 10u, Capacitor_SMD:C_0805_2012Metric, B.Cu at (170.9, 85.5)
- added C18: 22u, Capacitor_SMD:C_0805_2012Metric, B.Cu at (173.2, 75.6)
- added C19: 100n, Capacitor_SMD:C_0805_2012Metric, F.Cu at (141.1, 93.7)
- added C20: 100n, Capacitor_SMD:C_0805_2012Metric, F.Cu at (138.1, 91.2)
- added C21: 10u, Capacitor_SMD:C_0805_2012Metric, B.Cu at (149.3, 81.8)
- added C8: 100n, Capacitor_SMD:C_0805_2012Metric, B.Cu at (134.6, 90.4)
- added D13: SK6805, LED_SMD:LED_SK6805_PLCC4_2.4x2.7mm_P1.3mm, F.Cu at (142.4, 87.2)
- added D14: SK6805, LED_SMD:LED_SK6805_PLCC4_2.4x2.7mm_P1.3mm, F.Cu at (158.6, 87.4)
- added D15: SK6805, LED_SMD:LED_SK6805_PLCC4_2.4x2.7mm_P1.3mm, F.Cu at (155.5, 87.4)
- added D16: LED, LED_SMD:LED_0805_2012Metric, F.Cu at (115.5, 80.1)
- added D17: D_Schottky, Diode_SMD:D_0805_2012Metric, B.Cu at (176.2, 82.2)
- added D18: D_Schottky, Diode_SMD:D_0805_2012Metric, B.Cu at (176.2, 78.7)
- added D19: SP0504BAHT, Package_TO_SOT_SMD:SOT-23-5, B.Cu at (144.2, 76.2)
- added D2: LED, LED_SMD:LED_0805_2012Metric, F.Cu at (115.3, 103.3)
- added D20: SP0504BAHT, Package_TO_SOT_SMD:SOT-23-5, B.Cu at (126.5, 78.0)
- added D21: SP0504BAHT, Package_TO_SOT_SMD:SOT-23-5, B.Cu at (156.8, 78.0)
- added D22: PTVS12VZ1USK, Diode_SMD:Nexperia_DSN1608-2_1.6x0.8mm, B.Cu at (173.0, 102.2)
- added D23: PTVS12VZ1USK, Diode_SMD:Nexperia_DSN1608-2_1.6x0.8mm, B.Cu at (173.2, 97.1)
- added D24: PTVS12VZ1USK, Diode_SMD:Nexperia_DSN1608-2_1.6x0.8mm, B.Cu at (117.9, 121.2)
- added D25: PTVS12VZ1USK, Diode_SMD:Nexperia_DSN1608-2_1.6x0.8mm, B.Cu at (115.3, 114.0)
- added D26: PTVS5V0Z1USK, Diode_SMD:Nexperia_DSN1608-2_1.6x0.8mm, B.Cu at (148.7, 83.5)
- added D3: LED, LED_SMD:LED_0805_2012Metric, F.Cu at (115.3, 105.3)
- added G***: LOGO, frogs:frog_smallest, F.Cu at (163.5, 86.7)
- added G***: LOGO, frogs:frog_smallest, F.Cu at (128.5, 91.0)
- added J1: Conn_01x01_Pin, TestPoint:TestPoint_Pad_1.5x1.5mm, F.Cu at (141.2, 90.6)
- added R1: 10k, Resistor_SMD:R_0805_2012Metric, B.Cu at (119.0, 84.9)
- added TP11: 5v, TestPoint:TestPoint_Pad_D1.5mm, F.Cu at (171.3, 73.4)
- added U4: TXB0101DBV, Package_TO_SOT_SMD:SOT-23-6, F.Cu at (138.0, 93.9)
- added U5: AZ1117-5.0, Package_TO_SOT_SMD:SOT-223, B.Cu at (170.5, 80.3)
- C13, C14, R26, R27: moved to B.Cu
- C15, D4: moved to F.Cu
- D10, D11, D12, D9: value LED -> SK6805; footprint LED_SMD:LED_0805_2012Metric -> LED_SMD:LED_SK6805_PLCC4_2.4x2.7mm_P1.3mm
- J5: footprint Connector_PinSocket_2.54mm:PinSocket_1x03_P2.54mm_Vertical -> Connector_PinHeader_2.54mm:PinHeader_1x03_P2.54mm_Horizontal
- JP1: footprint Connector_PinHeader_2.54mm:PinHeader_1x03_P2.54mm_Vertical -> Jumper:SolderJumper-3_P1.3mm_Bridged2Bar12_RoundedPad1.0x1.5mm_NumberLabels; moved to B.Cu
- R32: value 500 -> 10k; moved to F.Cu
- SW1: footprint Button_Switch_THT:SW_CuK_OS102011MA1QN1_SPDT_Angled -> Button_Switch_THT:SW_Slide_SPDT_Angled_CK_OS102011MA1Q
- SW7, SW8: footprint Button_Switch_THT:SW_CuK_JS202011CQN_DPDT_Straight -> Button_Switch_THT:SW_E-Switch_EG1271_SPDT
- moved TP8 85.6 mm to (174.0, 121.5), turned to 90 degrees
- moved J2 76.8 mm to (136.7, 75.4)
- moved R30 62.9 mm to (173.3, 114.3), turned to 0 degrees
- moved R29 60.5 mm to (173.3, 110.1), turned to 180 degrees
- moved D5 60.5 mm to (173.3, 94.2), turned to 0 degrees
- moved D6 60.2 mm to (173.2, 92.1), turned to 180 degrees
- moved R21 60.2 mm to (170.9, 94.2), turned to 180 degrees
- moved R22 59.7 mm to (170.8, 92.1), turned to 180 degrees
- moved 1.1v1 59.2 mm to (175.9, 112.1), turned to 0 degrees
- moved R28 58.6 mm to (173.3, 106.1), turned to 0 degrees
- moved 2.2v1 57.5 mm to (175.9, 108.1), turned to 0 degrees
- moved D7 57.2 mm to (173.2, 89.9), turned to 180 degrees
- moved D8 56.9 mm to (173.2, 87.8), turned to 180 degrees
- moved R23 56.8 mm to (170.8, 89.9), turned to 180 degrees
- moved R31 56.5 mm to (170.8, 87.8), turned to 180 degrees
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Connections:
- D10 pad 1: Net-(D10-K) -> Net-(D10-DOUT)
- D10 pad 2: +3.3V -> GND
- D11 pad 1: Net-(D11-K) -> Net-(D11-DOUT)
- D11 pad 2: +3.3V -> GND
- D12 pad 2: +3.3V -> GND
- D9 pad 1: Net-(D9-K) -> Net-(D10-DIN)
- D9 pad 2: +3.3V -> GND
- J3 pad 1: /FUNCTION AMPLIFIER/CH1_OUT -> /FUNCTION AMPLIFIER/CH3_OUT
- J3 pad 3: /FUNCTION AMPLIFIER/CH4_OUT -> /FUNCTION AMPLIFIER/CH1_OUT
- J3 pad 7: /FUNCTION AMPLIFIER/CH3_OUT -> /FUNCTION AMPLIFIER/CH4_OUT
- J9 pad 2: /USART3_TX -> /USART3_CK
- J9 pad 4: /USART3_CK -> /USART3_TX
- JP1 pad 1: +12V -> VBUS
- JP1 pad 3: VBUS -> +12V
- R10 pad 2: Net-(U2B-+) -> Net-(U2D-+)
- R11 pad 1: Net-(U2A--) -> Net-(U2C--)
- R12 pad 1: Net-(U2B--) -> Net-(U2D--)
- R13 pad 1: /OPAMP1_VOUT -> /DAC1_OUT1
- R13 pad 2: Net-(U2C--) -> Net-(U2B--)
- R14 pad 2: Net-(U2C-+) -> Net-(U2B-+)
- R15 pad 1: /DAC1_OUT1 -> /OPAMP1_VOUT
- R15 pad 2: Net-(U2D--) -> Net-(U2A--)
- R16 pad 2: Net-(U2D-+) -> Net-(U2A-+)
- R17 pad 2: Net-(U2C-+) -> Net-(U2B-+)
- R18 pad 2: Net-(U2D-+) -> Net-(U2A-+)
- R19 pad 1: Net-(U2C--) -> Net-(U2B--)
- R20 pad 1: Net-(U2D--) -> Net-(U2A--)
- R32 pad 1: Net-(D9-K) -> /ENABLE
- R32 pad 2: /GPIO_4 -> GND
- R33 pad 1: Net-(D10-K) -> Net-(D16-K)
- R33 pad 2: /GPIO_2 -> GND
- R5 pad 1: /DAC1_OUT2 -> /OPAMP3_VOUT
- R5 pad 2: Net-(U2A--) -> Net-(U2C--)
- R6 pad 2: Net-(U2A-+) -> Net-(U2C-+)
- R7 pad 1: /OPAMP3_VOUT -> /DAC1_OUT2
- R7 pad 2: Net-(U2B--) -> Net-(U2D--)
- R8 pad 2: Net-(U2B-+) -> Net-(U2D-+)
- R9 pad 2: Net-(U2A-+) -> Net-(U2C-+)
- SW3 pad 3: /ADC1_IN5 -> /ADC1_IN4
- SW4 pad 3: /ADC2_IN12 -> /ADC1_IN5
- TP1 pad 1: /DAC1_OUT2 -> /OPAMP3_VOUT
- TP2 pad 1: /OPAMP3_VOUT -> /DAC1_OUT2
- U1 pad 11: /GPIO_4 -> /ADC1_IN4
- U1 pad 18: /ADC2_IN12 -> /DATA_IN
- U1 pad 2: /GPIO_1 -> unconnected-(U1-PC13-Pad2)
- U1 pad 3: /GPIO_2 -> /ENABLE
- U2 pad 1: /FUNCTION AMPLIFIER/CH1_OUT -> /FUNCTION AMPLIFIER/CH4_OUT
- U2 pad 14: /FUNCTION AMPLIFIER/CH4_OUT -> /FUNCTION AMPLIFIER/CH3_OUT
- U2 pad 7: /FUNCTION AMPLIFIER/CH3_OUT -> /FUNCTION AMPLIFIER/CH2_OUT
- U2 pad 8: /FUNCTION AMPLIFIER/CH2_OUT -> /FUNCTION AMPLIFIER/CH1_OUT
Routing:
- net VBUS: track 33.8 -> 113.2 mm, vias 2 -> 13
- net /NRST: track 2.75 -> 53.4 mm, vias 0 -> 3
- net /ADC2_IN4: track 6.50 -> 46.9 mm
- net /ADC2_IN12: track 37.1 -> 0.00 mm
- net /ADC1_IN4: track 0.00 -> 32.8 mm, vias 0 -> 1
- net /GPIO_IN1: track 56.8 -> 24.8 mm, vias 0 -> 1
- net /ADC2_IN3: track 8.13 -> 39.7 mm
- net /USART3_CK: track 0.00 -> 30.3 mm
- net +3.3V: track 44.4 -> 68.8 mm, vias 27 -> 25
- net /USART3_TX: track 17.8 -> 41.5 mm
- net /debug_led1: track 3.88 -> 24.3 mm, vias 0 -> 1
- net Net-(D4-A): track 3.30 -> 22.7 mm, vias 0 -> 1
- net /ENABLE: track 0.00 -> 18.9 mm, vias 0 -> 2
- net /GPIO_2: track 18.8 -> 0.00 mm
- net /debug_led2: track 4.66 -> 23.4 mm, vias 0 -> 1
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Other:
- board size 71 x 60.9 mm -> 64 x 56 mm
- board text added: "3&4 >"
- board text added: "3.3V"
- board text added: "< 1&2"
- board text added: "AZ1117-3v3"
- board text added: "B"
- board text added: "B : busy G : good R : error"
- board text added: "BOOT-PROG"
- board text added: "C"
- board text added: "CH1"
- board text added: "CH2"
- board text added: "CH3"
- board text added: "CH4"
- board text added: "CHANNEL_LINKS"
- board text added: "CLK"
- board text added: "D"
- board text added: "DEBUG LEDS"
- board text added: "DESGINED BY"
- board text added: "DONT FROGET ABOUT IT"
- board text added: "FREQ.1"
- board text added: "FREQ.2"
- board text added: "FREQ.3"
- board text added: "FREQ.4"
- board text added: "FUALT"
- board text added: "I2S_CLK"
- board text added: "I2S_SD"
- board text added: "LED.1"
- board text added: "LED.2"
- board text added: "LINK"
- board text added: "MOSTLY"
- board text added: "PHASE.1"
- board text added: "PHASE.2"
- board text added: "PROG MODE"
- board text added: "STATUS LEDS"
- board text added: "STM32G431CBTx"
- board text added: "SWD_TRACE"
- board text added: "THE RAT KING"
- board text added: "USART"
- board text added: "USB TYPE C"
- board text added: "USB_STATUS"
- board text added: "WILLIAM"
- board text added: "Y"
- board text added: "YOU JUST GOT FROGGED"
- board text removed: "+"
- board text removed: "-"
- board text removed: "1"
- board text removed: "1.1v"
- board text removed: "10k"
- board text removed: "12v--USB"
- board text removed: "13K"
- board text removed: "2"
- board text removed: "2.2v"
- board text removed: "3"
- board text removed: "4"
- board text removed: "91k"
- board text removed: "ADC"
- board text removed: "AMP CONFIG"
- board text removed: "AMPLIFER"
- board text removed: "CHANNEL 1 !link - FREQ link - PHASE"
- board text removed: "CHANNEL 2 !link - FREQ link - FREQ"
- board text removed: "CHANNEL 3 !link - FREQ link - PHASE"
- board text removed: "CHANNEL 4 !link - FREQ link - FREQ"
- board text removed: "CHANNEL_1_WAVEFORM"
- board text removed: "CHANNEL_2_WAVEFORM"
- board text removed: "CHANNEL_3_WAVEFORM"
- board text removed: "CHANNEL_4_WAVEFORM"
- board text removed: "CHANNEL_LINK_1-2"
- board text removed: "CHANNEL_LINK_3-4"
- board text removed: "CK"
- board text removed: "DNP"
- board text removed: "F"
- board text removed: "FLASH--PROG"
- board text removed: "I2S_CK"
- board text removed: "IS2_SD"
- board text removed: "LED_1"
- board text removed: "LED_2"
- board text removed: "MNT M3"
- board text removed: "O"
- board text removed: "OSC_DNP use internal"
- board text removed: "R1"
- board text removed: "R2"
- board text removed: "R3"
- board text removed: "R4"
- board text removed: "REV3-pending"
- board text removed: "SIG OUT"
- board text removed: "SIG_IN"
- board text removed: "SIG_OUT"
- board text removed: "STM32G431CBT6"
- board text removed: "TL074"
- board text removed: "USB-TYPE-C"
- board text removed: "WAVEFORM SELECT"
- board text removed: "channel linking allows 2 output channels to be link together they share the same frequency but can have differnt phases. to change the freq use the pot marked link-FREQ and change the phase use the pot marked link-PHASE"
- board text removed: "have you touched grass today"
- board text removed: "mostly desgined by william"
- board text removed: "the rat king will rise again"
- board text removed: "this will only give a sig with 0 DC if VPWR is > ±12v"
- board text removed: "to change the freq of a channel use the pot marked !link - FREQ"
- board text removed: "to change the wave form use the slide switch"
- board text removed: "±12v"
